File: hardware/Main_Board.sch (EAGLE design)
At the start: 52 parts, among them Q1 CSD87313DMS, Q2 CSD16406Q3, U1 BQ24210, U2 BQ29733DSER, U3 LP38693MPX-ADJ/NOPB, U4 ESP-WROOM-02D, U5 INA219AID, U6 TC78H630FNG/TSSOP16, U7 LT1716

Commit message: Update docs for Rev 1.1B changes
Parts:
- added R16: 10KΩ, rcl:R-US_R0805
- added RST: PTS636_SL43_SMTR_LFS, Genericor Parts:PTS636_SL43_SMTR_LFS
- C1: device rcl:CPOL-USE7.5-16 -> Genericor Parts:CPOL-7.62-18-27
- renumbered BOOT to FLASH
Connections:
- net DRV_1: now also FLASH.2, R11.2
- net DRV_2: now also R16.1; no longer FLASH.2, R11.2
- net EN-RST: now also RST.2
- net GND: now also R16.2, RST.1
Other:
- note added: "1.1B"
- note removed: "1.0A"
- moved on the sheet: C6, R12
